Commit message: ur5 scan movement 수정

File: moveit2_ws/src/ur5e_laser_moveit_config/urdf/ur5e_laser.urdf.xacro (robot description, xacro)
@@ -5,8 +5,10 @@
     Hand-eye convention used by the application:
       ^tool0 T_sensor =
-        [-1  0  0    0 mm ]
-        [ 0  1  0    0 mm ]
+        [ 1  0  0    0 mm ]
+        [ 0 -1  0    0 mm ]
         [ 0  0 -1  151 mm ]
         [ 0  0  0    1    ]
+    This includes the physical 180-degree sensor rotation about the final
+    wrist_3/tool0 +Z rotation axis.
       ^sensor T_physical = Trans(0, 0, +80 mm)
     The official UR model has the fixed axis relationship
@@ -16,5 +18,5 @@
     Therefore the same physical mounting is encoded here directly as
       ^flange p_sensor = [151, 0, 0] mm
-      ^flange R_sensor = RPY(+90 deg, 0, -90 deg)
+      ^flange R_sensor = RPY(-90 deg, 0, +90 deg)
     This keeps the physical attachment expressed from `flange`, while the
     application may continue to store T_tcp_sensor with `tcp == tool0`.
@@ -86,5 +88,5 @@
     <parent link="flange"/>
     <child link="sensor_measurement_frame"/>
-    <origin xyz="0.151 0 0" rpy="1.57079632679 0 -1.57079632679"/>
+    <origin xyz="0.151 0 0" rpy="-1.57079632679 0 1.57079632679"/>
   </joint>
   <!-- P is the physical reference point used by pose generation/planning. -->

File: moveit2_ws/src/ur5e_laser_visualization/urdf/ur5e_ljv7080_preview.urdf.xacro (robot description, xacro)
@@ -5,8 +5,10 @@
     Coordinate convention used here:
       ^tool0 T_sensor =
-        [-1  0  0    0 mm ]
-        [ 0  1  0    0 mm ]
+        [ 1  0  0    0 mm ]
+        [ 0 -1  0    0 mm ]
         [ 0  0 -1  151 mm ]
         [ 0  0  0    1    ]
+    This includes the physical 180-degree sensor rotation about the final
+    wrist_3/tool0 +Z rotation axis.
       ^sensor T_physical = Trans(0, 0, +80 mm)
     The official UR ROS model has
@@ -16,5 +18,5 @@
     Therefore the same sensor mounting is
       ^flange p_sensor = [151, 0, 0] mm
-      ^flange R_sensor = RPY(+90 deg, 0, -90 deg).
+      ^flange R_sensor = RPY(-90 deg, 0, +90 deg).
   -->
   <xacro:include filename="$(find ur_description)/urdf/ur_macro.xacro"/>
@@ -83,5 +85,5 @@
     <child link="sensor_measurement_frame"/>
     <!-- ^flange T_sensor: +151 mm along +X_flange. -->
-    <origin xyz="0.151 0 0" rpy="1.57079632679 0 -1.57079632679"/>
+    <origin xyz="0.151 0 0" rpy="-1.57079632679 0 1.57079632679"/>
   </joint>
   <xacro:frame_triad name="sensor_axes_preview" parent="sensor_measurement_frame" origin_rgba="1.0 0.05 0.85 1"/>
